File: PW-2.kicad_sch (KiCad schematic)
At the start: 6 parts

Commit message: some
Parts:
- added C? (x4): C, symbol Device:C
- added D?: D, symbol Device:D
- added F?: Fuse, symbol Device:Fuse
- added FL?: BNX025, Filter:Filter_Murata_BNX025, symbol Filter:BNX025
- added R? (x5): R, symbol Device:R
- added U?: NCP1034, Package_SO:SOIC-16_3.9x9.9mm_P1.27mm, symbol Regulator_Switching_additional:NCP1034
- added U?: L7812, symbol Regulator_Linear:L7812
Connections:
- net +BATT: now also F?.1
- net GNDPWR: now also FL?.3 (PSG)
- new net: R?.2, U?.1 (OCSET)
- new net: C?.1, FL?.2 (CB), R?.2, U?.1 (IN)
- new net: R?.1, R?.2, U?.16 (UVLO)
- new net: R?.2, U?.15 (RT)
- new net: R?.2, U?.5 (SYNC)
- new net: C?.1, D?.1 (K), U?.9 (VB)
- new net: C?.1, D?.2 (A), U?.12 (VCC), U?.3 (OUT), U?.8 (DRVCCC)
- new net: C?.2, U?.11 (VS)
- new net: C?.1, U?.4 (SS/~{SD})
- new net: F?.2, FL?.1 (B)
- new net GND: C?.2, C?.2, C?.2, FL?.4 (CG), R?.1, R?.1, R?.1, R?.1, U?.14 (GND), U?.2 (GND), U?.6 (PGND)
