File: 12-19V_supply.kicad_sch (KiCad schematic)
At the start: 0 parts

Commit message: little change
Parts:
- added C? (x7): C, symbol Device:C
- added C? (x2): C_Polarized, symbol Device:C_Polarized
- added D?: D, symbol Device:D
- added L?: L, symbol Device:L
- added Q? (x2): TPH11006NL, Package_SON_additional:Toshiba_SOP_Advance, symbol Transistor_FET_additional:TPH11006NL
- added R? (x10): R, symbol Device:R
- added U?: L7812, symbol Regulator_Linear:L7812
- added U?: NCP1034, Package_SO:SOIC-16_3.9x9.9mm_P1.27mm, symbol Regulator_Switching_additional:NCP1034
Connections:
- new net: C?.1, D?.1 (K), U?.9 (VB)
- new net: C?.2, L?.1, Q?.1 (S), Q?.2 (S), Q?.3 (S), Q?.5 (D), Q?.6 (D), Q?.7 (D), Q?.8 (D), R?.2, U?.11 (VS)
- new net: C?.1, R?.1, U?.3 (COMP)
- new net: C?.1, C?.2, C?.2, R?.1, R?.2, U?.2 (FB)
- new net: Q?.4 (G), U?.10 (HDRV)
- new net: R?.1, R?.2, U?.16 (UVLO)
- new net: R?.2, U?.1 (OCSET)
- new net: C?.2, R?.2
- new net: R?.2, U?.5 (SYNC)
- new net: C?.1, R?.2
- new net: C?.1, U?.4 (SS/~{SD})
- new net: C?.1, D?.2 (A), U?.12 (VCC), U?.3 (OUT), U?.8 (DRVCCC)
- new net: Q?.4 (G), U?.7 (LDRV)
- new net: R?.1, U?.13 (OCIN)
- new net: R?.2, U?.15 (RT)
- new net 12-19V_out: C?.1, C?.1, L?.2, R?.1, R?.1
- new net 24V_supply: C?.1, Q?.5 (D), Q?.6 (D), Q?.7 (D), Q?.8 (D), R?.2, U?.1 (IN)
- new net GND: C?.2, C?.2, C?.2, C?.2, C?.2, Q?.1 (S), Q?.2 (S), Q?.3 (S), R?.1, R?.1, R?.1, R?.1, R?.2, U?.14 (GND), U?.2 (GND), U?.6 (PGND)
